Commit message: added server action detection

File: franka_ros/franka_description/robots/common/franka_arm.xacro (robot description, xacro)
@@ -128,5 +128,5 @@
       <parent link="${arm_id}_link9"/>
       <child link="${arm_id}_link10"/>
-      <origin rpy=" 0 ${pi/2} 0" xyz="0.1 0 0.0"/>
+      <origin rpy=" 0 ${pi/2} 0" xyz="0.0 0 0.0"/>
     </joint>
      <gazebo reference="${arm_id}_link10">
